File: TXB0104 Level translator.sch (KiCad schematic (older format))
At the start: 6 parts, among them P1 CONN_7, P2 CONN_7, U1 TXB0104

Commit message: Ready for manufacturing
Parts:
- gave numbers to parts that had none: 1
Connections:
- net +3.3VP: no longer P1.6 (P6)
- net +5V: no longer P2.6 (P6)
- net GND: now also P1.2 (P2), P2.2 (P2); no longer P1.7 (P7)
- net at U1.10 (B4_): now also P2.6 (P6); no longer P2.5 (P5)
- net at U1.11 (B3): now also P2.5 (P5); no longer P2.4 (P4)
- net at U1.12 (B2): now also P2.4 (P4); no longer P2.3 (P3)
- net at U1.13 (B1): now also P2.3 (P3); no longer P2.2 (P2)
- net at U1.2 (A1): now also P1.3 (P3); no longer P1.2 (P2)
- net at U1.3 (A2): now also P1.4 (P4); no longer P1.3 (P3)
- net at U1.4 (A3): now also P1.5 (P5); no longer P1.4 (P4)
- net at U1.5 (A4): now also P1.6 (P6); no longer P1.5 (P5)
- net OE: now reaches JP1.1, P2.7 (P7), U1.8 (OE)
- net OE: now also P1.7 (P7)
Changed lines of the file:
@@
 	-1   0    0    -1
 $EndComp
-Wire Wire Line
-	4000 3600 4000 3450
-Wire Wire Line
-	4000 3450 5000 3450
-Wire Wire Line
-	4000 3700 4150 3700
-Wire Wire Line
-	4150 3700 4150 3650
-Wire Wire Line
-	4150 3650 5000 3650
-Wire Wire Line
-	4000 3800 5000 3800
-Wire Wire Line
-	5000 3800 5000 3850
-Wire Wire Line
-	4000 3900 5000 3900
-Wire Wire Line
-	5000 3900 5000 4000
-Wire Wire Line
-	4000 4200 4000 4450
-Wire Wire Line
-	4000 4450 5000 4450
-Wire Wire Line
-	4000 4000 4250 4000
-Wire Wire Line
-	4250 4000 4250 4150
-Wire Wire Line
-	4250 4150 5000 4150
-Wire Wire Line
-	6300 3450 7300 3450
-Wire Wire Line
-	7300 3450 7300 3600
-Wire Wire Line
-	6300 3650 7200 3650
-Wire Wire Line
-	7200 3650 7200 3700
-Wire Wire Line
-	7200 3700 7300 3700
-Wire Wire Line
-	6300 3850 6300 3800
-Wire Wire Line
-	6300 3800 7300 3800
-Wire Wire Line
-	6300 4000 6400 4000
-Wire Wire Line
-	6400 4000 6400 3900
-Wire Wire Line
-	6400 3900 7300 3900
-Wire Wire Line
-	6300 4150 6500 4150
-Wire Wire Line
-	6500 4150 6500 4000
-Wire Wire Line
-	6500 4000 7300 4000
-Wire Wire Line
-	6300 4450 7300 4450
-Wire Wire Line
-	7300 4450 7300 4200
 $Comp
 L C C2
@@
 	1    0    0    -1
 $EndComp
-Wire Wire Line
-	6500 2740 6500 3450
-Connection ~ 6500 3450
-Wire Wire Line
-	6900 3050 7100 3050
-Wire Wire Line
-	7100 3050 7100 3200
-Wire Wire Line
-	4850 2800 4850 3450
-Connection ~ 4850 3450
 $Comp
 L GND #PWR02
@@
 	1    0    0    -1
 $EndComp
-Wire Wire Line
-	4450 3050 4200 3050
-Wire Wire Line
-	4200 3050 4200 3200
-Wire Bus Line
-	2850 2350 8300 2350
-Wire Bus Line
-	8300 2350 8300 5500
-Wire Bus Line
-	8300 5500 2850 5500
-Wire Bus Line
-	2850 5500 2850 2350
 Text Notes 3750 2600 0    60   ~ 12
 Bidirectional Level translator
@@
 	1    0    0    -1
 $EndComp
-Connection ~ 4850 4450
-Connection ~ 6700 4450
-$Comp
-L +3.3VP #PWR?
+$Comp
+L +3.3VP #PWR04
 U 1 1 554364B2
 P 4850 2800
-F 0 "#PWR?" H 4900 2830 20  0001 C CNN
+F 0 "#PWR04" H 4900 2830 20  0001 C CNN
 F 1 "+3.3VP" H 4850 2890 30  0000 C CNN
 F 2 "" H 4850 2800 60  0000 C CNN
@@
 	1    0    0    -1
 $EndComp
-Connection ~ 4850 3050
-$Comp
-L +5V #PWR?
+$Comp
+L +5V #PWR05
 U 1 1 554364F4
 P 6500 2740
-F 0 "#PWR?" H 6500 2830 20  0001 C CNN
+F 0 "#PWR05" H 6500 2830 20  0001 C CNN
 F 1 "+5V" H 6500 2830 30  0000 C CNN
 F 2 "" H 6500 2740 60  0000 C CNN
@@
 	1    0    0    -1
 $EndComp
-Connection ~ 6500 3050
-Wire Wire Line
-	4000 4100 4160 4100
-Wire Wire Line
-	4160 4100 4160 4310
-Wire Wire Line
-	4160 4310 4580 4310
-Wire Wire Line
-	4580 4310 4580 3450
-Connection ~ 4580 3450
-$Comp
-L +3.3VP #PWR?
+$Comp
+L +3.3VP #PWR06
 U 1 1 55436701
 P 7900 4510
-F 0 "#PWR?" H 7950 4540 20  0001 C CNN
+F 0 "#PWR06" H 7950 4540 20  0001 C CNN
 F 1 "+3.3VP" H 7900 4600 30  0000 C CNN
 F 2 "" H 7900 4510 60  0000 C CNN
@@
 $EndComp
 $Comp
-L BREAKER JP?
+L BREAKER JP1
 U 1 1 55436743
 P 7280 4750
-F 0 "JP?" H 7280 4700 50  0000 C CNN
+F 0 "JP1" H 7280 4700 50  0000 C CNN
 F 1 "Jumper" H 7280 4600 50  0000 C CNN
 F 2 "~" H 7280 4750 60  0000 C CNN
@@
 	1    0    0    -1
 $EndComp
-Wire Wire Line
-	6780 4750 6700 4750
-Wire Wire Line
-	6700 4750 6700 4450
-Wire Wire Line
-	7900 4510 7900 4750
-Wire Wire Line
-	7900 4750 7780 4750
-Wire Wire Line
-	7300 4100 6710 4100
-Wire Wire Line
-	6710 4100 6710 3450
-Connection ~ 6710 3450
-Wire Wire Line
-	4850 4680 4850 4450
 Text Notes 4160 5000 0    60   ~ 12
 VCCA 1.2V to 3.6V
@@
 NoConn ~ 6300 4300
 NoConn ~ 5000 4300
+Wire Wire Line
+	4000 3600 4000 3450
+Wire Wire Line
+	4000 3450 5000 3450
+Wire Wire Line
+	6300 3450 7300 3450
+Wire Wire Line
+	7300 3450 7300 3600
+Wire Wire Line
+	6300 4450 7300 4450
+Wire Wire Line
+	7300 4450 7300 4200
+Wire Wire Line
+	6500 2740 6500 3450
+Connection ~ 6500 3450
+Wire Wire Line
+	6900 3050 7100 3050
+Wire Wire Line
+	7100 3050 7100 3200
+Wire Wire Line
+	4850 2800 4850 3450
+Connection ~ 4850 3450
+Wire Wire Line
+	4450 3050 4200 3050
+Wire Wire Line
+	4200 3050 4200 3200
+Wire Bus Line
+	2850 2350 8300 2350
+Wire Bus Line
+	8300 2350 8300 5500
+Wire Bus Line
+	8300 5500 2850 5500
+Wire Bus Line
+	2850 5500 2850 2350
+Connection ~ 6700 4450
+Connection ~ 4850 3050
+Connection ~ 6500 3050
+Connection ~ 4580 3450
+Wire Wire Line
+	6780 4750 6700 4750
+Wire Wire Line
+	6700 4750 6700 4450
+Wire Wire Line
+	7900 4510 7900 4750
+Wire Wire Line
+	7900 4750 7780 4750
+Wire Wire Line
+	4850 4680 4850 4450
+Wire Wire Line
+	4220 4450 5000 4450
+Wire Wire Line
+	4000 3800 4440 3800
+Wire Wire Line
+	4440 3800 4440 3650
+Wire Wire Line
+	4440 3650 5000 3650
+Wire Wire Line
+	4000 3900 4570 3900
+Wire Wire Line
+	4570 3900 4570 3850
+Wire Wire Line
+	4570 3850 5000 3850
+Wire Wire Line
+	4000 4000 5000 4000
+Wire Wire Line
+	4000 4100 4650 4100
+Wire Wire Line
+	4650 4100 4650 4150
+Wire Wire Line
+	4650 4150 5000 4150
+Text Label 4000 4200 0    60   ~ 0
+OE
+Text Label 6520 4450 0    60   ~ 0
+OE
+Wire Wire Line
+	4000 3700 4220 3700
+Wire Wire Line
+	4220 3700 4220 4450
+Connection ~ 4850 4450
+Wire Wire Line
+	6300 3650 6940 3650
+Wire Wire Line
+	6940 3650 6940 3800
+Wire Wire Line
+	6940 3800 7300 3800
+Wire Wire Line
+	6300 3850 6820 3850
+Wire Wire Line
+	6820 3850 6820 3900
+Wire Wire Line
+	6820 3900 7300 3900
+Wire Wire Line
+	6300 4000 7300 4000
+Wire Wire Line
+	6300 4150 6830 4150
+Wire Wire Line
+	6830 4150 6830 4100
+Wire Wire Line
+	6830 4100 7300 4100
+$Comp
+L GND #PWR07
+U 1 1 55824F86
+P 7060 3540
+F 0 "#PWR07" H 7060 3290 60  0001 C CNN
+F 1 "GND" H 7060 3390 60  0000 C CNN
+F 2 "" H 7060 3540 60  0000 C CNN
+F 3 "" H 7060 3540 60  0000 C CNN
+	1    7060 3540
+	1    0    0    -1
+$EndComp
+Wire Wire Line
+	7060 3540 7230 3540
+Wire Wire Line
+	7230 3540 7230 3700
+Wire Wire Line
+	7230 3700 7300 3700
 $EndSCHEMATC
